File: a2card_template.sch (KiCad schematic (older format))
At the start: 1 part

Commit message: Landed the Leako PLCC Z80
Parts:
- added U10: PLCCZ80, Package_LCC:PLCC-44_THT-Socket, symbol LeadedSolder:PLCCZ80
Changed lines of the file:
@@
+	1    0    0    -1
+$EndComp
+$Comp
+L LeadedSolder:PLCCZ80 U10
+U 1 1 61560785
+P 7025 1925
+F 0 "U10" H 7025 2040 50  0000 C CNN
+F 1 "PLCCZ80" H 7025 1949 50  0000 C CNN
+F 2 "Package_LCC:PLCC-44_THT-Socket" H 7025 1925 50  0001 C CNN
+F 3 "" H 7025 1925 50  0001 C CNN
+	1    7025 1925
 	1    0    0    -1
 $EndComp

Commit message: Filling in the schemaitc
Parts:
- added U14, U16, U17: 74LS367, Package_DIP:DIP-16_W7.62mm, symbol 74xx:74LS367
Connections:
- net labels added: +5V, GND, a0, a0', a1, a1', a10, a10', a11, a11', a12, a12', a13, a13', a14, a14', a15, a15', a2, a2', a3, a3', a4, a4', a5, a5', a6, a6', a7, a7', a8, a8', a9, a9', d0, d1, d2, d3, d4, d5, d6, d7
- wire segments 0 -> 12
Other:
- note added: "TODO: Figure out enables"
- moved on the sheet: BUS1

Commit message: Add data-bus latch
Parts:
- added U1: 74LS373, Package_DIP:DIP-20_W7.62mm, symbol 74xx:74LS373
Connections:
- net labels added: d0', d1', d2', d3', d4', d5', d6', d7', ~RD, ø0
- wire segments 12 -> 13
Other:
- note added: "TODO: Don't be afraid to reorder these so they make an easier route"
Changed lines of the file:
@@
 Text Label 925  4825 2    50   ~ 0
 d7
+$Comp
+L 74xx:74LS373 U1
+U 1 1 6158A69D
+P 10375 5150
+F 0 "U1" H 10375 6131 50  0000 C CNN
+F 1 "74LS373" H 10375 6040 50  0000 C CNN
+F 2 "Package_DIP:DIP-20_W7.62mm" H 10375 5150 50  0001 C CNN
+F 3 "http://www.ti.com/lit/gpn/sn74LS373" H 10375 5150 50  0001 C CNN
+F 4 "296-1660-5-ND‎" H 10375 5150 50  0001 C CNN "DigiKey"
+	1    10375 5150
+	-1   0    0    -1
+$EndComp
+Text Label 10875 4750 0    50   ~ 0
+d0
+Text Label 10875 4650 0    50   ~ 0
+d1
+Text Label 10875 4850 0    50   ~ 0
+d7
+Text Label 10875 4950 0    50   ~ 0
+d2
+Text Label 10875 5050 0    50   ~ 0
+d6
+Text Label 10875 5150 0    50   ~ 0
+d5
+Text Label 10875 5250 0    50   ~ 0
+d3
+Text Label 10875 5350 0    50   ~ 0
+d4
+Text Notes 8450 6450 0    50   ~ 0
+TODO: Don't be afraid to reorder these so they make an easier route
+$Comp
+L power:GND #PWR0111
+U 1 1 6158F491
+P 10375 5950
+F 0 "#PWR0111" H 10375 5700 50  0001 C CNN
+F 1 "GND" H 10380 5777 50  0000 C CNN
+F 2 "" H 10375 5950 50  0001 C CNN
+F 3 "" H 10375 5950 50  0001 C CNN
+	1    10375 5950
+	1    0    0    -1
+$EndComp
+$Comp
+L power:+5V #PWR0112
+U 1 1 6158FC8D
+P 10600 4350
+F 0 "#PWR0112" H 10600 4200 50  0001 C CNN
+F 1 "+5V" H 10615 4523 50  0000 C CNN
+F 2 "" H 10600 4350 50  0001 C CNN
+F 3 "" H 10600 4350 50  0001 C CNN
+	1    10600 4350
+	1    0    0    -1
+$EndComp
+Wire Wire Line
+	10600 4350 10375 4350
+Text Label 10875 5550 0    50   ~ 0
+ø0
+Text Label 925  4425 2    50   ~ 0
+ø0
+Text Label 10875 5650 0    50   ~ 0
+~RD
+Text Label 7525 3575 0    50   ~ 0
+~RD
+Text Label 9875 4650 2    50   ~ 0
+d1'
+Text Label 9875 4750 2    50   ~ 0
+d0'
+Text Label 9875 4850 2    50   ~ 0
+d7'
+Text Label 9875 4950 2    50   ~ 0
+d2'
+Text Label 9875 5050 2    50   ~ 0
+d6'
+Text Label 9875 5150 2    50   ~ 0
+d5'
+Text Label 9875 5250 2    50   ~ 0
+d3'
+Text Label 9875 5350 2    50   ~ 0
+d4'
+Text Label 7525 2125 0    50   ~ 0
+d0'
+Text Label 7525 2225 0    50   ~ 0
+d1'
+Text Label 7525 2325 0    50   ~ 0
+d2'
+Text Label 7525 2425 0    50   ~ 0
+d3'
+Text Label 7525 2525 0    50   ~ 0
+d4'
+Text Label 7525 2625 0    50   ~ 0
+d5'
+Text Label 7525 2725 0    50   ~ 0
+d6'
+Text Label 7525 2825 0    50   ~ 0
+d7'
 $EndSCHEMATC

Commit message: Fix reference for U15
Parts:
- renumbered U1 to U15
Changed lines of the file:
@@
 d7
 $Comp
-L 74xx:74LS373 U1
+L 74xx:74LS373 U15
 U 1 1 6158A69D
 P 10375 5150
-F 0 "U1" H 10375 6131 50  0000 C CNN
+F 0 "U15" H 10375 6131 50  0000 C CNN
 F 1 "74LS373" H 10375 6040 50  0000 C CNN
 F 2 "Package_DIP:DIP-20_W7.62mm" H 10375 5150 50  0001 C CNN

Commit message: Configuration DIP
Parts:
- added RN9: 10kΩ, Resistor_THT:R_Array_SIP5, symbol Device:R_Network04_US
- added S1: SW_DIP_x04, Button_Switch_THT:SW_DIP_SPSTx04_Slide_9.78x12.34mm_W7.62mm_P2.54mm, symbol Switch:SW_DIP_x04
Connections:
- net labels added: ~IRQ, ~NMI, ~Z80_IRQ, ~Z80_NMI
- wire segments 13 -> 21
Changed lines of the file:
@@
 Text Label 7525 2825 0    50   ~ 0
 d7'
+$Comp
+L Switch:SW_DIP_x04 S1
+U 1 1 61569342
+P 9975 1425
+F 0 "S1" H 9975 1892 50  0000 C CNN
+F 1 "SW_DIP_x04" H 9975 1801 50  0000 C CNN
+F 2 "Button_Switch_THT:SW_DIP_SPSTx04_Slide_9.78x12.34mm_W7.62mm_P2.54mm" H 9975 1425 50  0001 C CNN
+F 3 "~" H 9975 1425 50  0001 C CNN
+	1    9975 1425
+	-1   0    0    -1
+$EndComp
+Text Label 9675 1425 2    50   ~ 0
+~NMI
+Text Label 10850 1425 0    50   ~ 0
+~Z80_NMI
+Text Label 7725 3175 0    50   ~ 0
+~Z80_NMI
+Wire Wire Line
+	7725 3175 7525 3175
+Text Label 925  2225 2    50   ~ 0
+~NMI
+$Comp
+L Device:R_Network04_US RN9
+U 1 1 6156C017
+P 10600 925
+F 0 "RN9" H 10788 971 50  0000 L CNN
+F 1 "10kΩ" H 10788 880 50  0000 L CNN
+F 2 "Resistor_THT:R_Array_SIP5" V 10875 925 50  0001 C CNN
+F 3 "http://www.vishay.com/docs/31509/csc.pdf" H 10600 925 50  0001 C CNN
+	1    10600 925
+	1    0    0    -1
+$EndComp
+$Comp
+L power:+5V #PWR0113
+U 1 1 6156D36C
+P 10400 725
+F 0 "#PWR0113" H 10400 575 50  0001 C CNN
+F 1 "+5V" H 10415 898 50  0000 C CNN
+F 2 "" H 10400 725 50  0001 C CNN
+F 3 "" H 10400 725 50  0001 C CNN
+	1    10400 725
+	1    0    0    -1
+$EndComp
+Wire Wire Line
+	10275 1425 10600 1425
+Text Label 9675 1525 2    50   ~ 0
+~IRQ
+Text Label 10850 1525 0    50   ~ 0
+~Z80_IRQ
+Wire Wire Line
+	10850 1525 10700 1525
+Wire Wire Line
+	10700 1125 10700 1525
+Connection ~ 10700 1525
+Wire Wire Line
+	10700 1525 10275 1525
+Wire Wire Line
+	10600 1125 10600 1425
+Connection ~ 10600 1425
+Wire Wire Line
+	10600 1425 10850 1425
+Text Label 925  2425 2    50   ~ 0
+~IRQ
+Text Label 7725 3075 0    50   ~ 0
+~Z80_IRQ
+Wire Wire Line
+	7725 3075 7525 3075
 $EndSCHEMATC

Commit message: Popping more junk
Parts:
- added R13: 10kΩ, Resistor_THT:R_Array_SIP9, symbol Device:R_Network08_US
- added U9: 74LS367, Package_DIP:DIP-16_W7.62mm, symbol 74xx:74LS367
Connections:
- net labels added: 7M, DMA_IN, INT_IN_OUT, ~BUSRQ
- wire segments 21 -> 34
Other:
- note added: "TODO: 7M"
- note added: "TODO: U3"
- note added: "TODO: ø1"
Changed lines of the file:
@@
 Wire Wire Line
 	7725 3075 7525 3075
+Text Label 2525 2025 0    50   ~ 0
+INT_IN_OUT
+Text Label 925  2025 2    50   ~ 0
+INT_IN_OUT
+$Comp
+L 74xx:74LS367 U9
+U 1 1 6157726E
+P 10275 2550
+F 0 "U9" H 10275 3431 50  0000 C CNN
+F 1 "74LS367" H 10275 3340 50  0000 C CNN
+F 2 "Package_DIP:DIP-16_W7.62mm" H 10275 2550 50  0001 C CNN
+F 3 "http://www.ti.com/lit/gpn/sn74LS367" H 10275 2550 50  0001 C CNN
+F 4 "296-3701-5-ND‎" H 10275 2550 50  0001 C CNN "DigiKey"
+	1    10275 2550
+	1    0    0    -1
+$EndComp
+$Comp
+L power:+5V #PWR0114
+U 1 1 615799C2
+P 10525 1850
+F 0 "#PWR0114" H 10525 1700 50  0001 C CNN
+F 1 "+5V" H 10540 2023 50  0000 C CNN
+F 2 "" H 10525 1850 50  0001 C CNN
+F 3 "" H 10525 1850 50  0001 C CNN
+	1    10525 1850
+	1    0    0    -1
+$EndComp
+Wire Wire Line
+	10525 1850 10275 1850
+$Comp
+L power:GND #PWR0115
+U 1 1 6157A62A
+P 10275 3250
+F 0 "#PWR0115" H 10275 3000 50  0001 C CNN
+F 1 "GND" H 10280 3077 50  0000 C CNN
+F 2 "" H 10275 3250 50  0001 C CNN
+F 3 "" H 10275 3250 50  0001 C CNN
+	1    10275 3250
+	1    0    0    -1
+$EndComp
+Text Label 10775 2450 0    50   ~ 0
+d7
+Text Label 10775 2350 0    50   ~ 0
+d6
+Text Label 10775 2250 0    50   ~ 0
+d5
+Text Label 10775 2150 0    50   ~ 0
+d4
+Text Label 9775 2450 2    50   ~ 0
+d7'
+Text Label 9775 2350 2    50   ~ 0
+d6'
+Text Label 9775 2250 2    50   ~ 0
+d5'
+Text Label 9775 2150 2    50   ~ 0
+d4'
+$Comp
+L Device:R_Network08_US R13
+U 1 1 6157F8C6
+P 8250 1750
+F 0 "R13" H 8638 1796 50  0000 L CNN
+F 1 "10kΩ" H 8638 1705 50  0000 L CNN
+F 2 "Resistor_THT:R_Array_SIP9" V 8725 1750 50  0001 C CNN
+F 3 "http://www.vishay.com/docs/31509/csc.pdf" H 8250 1750 50  0001 C CNN
+	1    8250 1750
+	1    0    0    -1
+$EndComp
+$Comp
+L power:+5V #PWR0116
+U 1 1 61580C5A
+P 7850 1550
+F 0 "#PWR0116" H 7850 1400 50  0001 C CNN
+F 1 "+5V" H 7865 1723 50  0000 C CNN
+F 2 "" H 7850 1550 50  0001 C CNN
+F 3 "" H 7850 1550 50  0001 C CNN
+	1    7850 1550
+	1    0    0    -1
+$EndComp
+Text Label 8450 1950 3    50   ~ 0
+d7'
+Text Label 8350 1950 3    50   ~ 0
+d5'
+Text Label 8250 1950 3    50   ~ 0
+d0'
+Text Label 8150 1950 3    50   ~ 0
+d3'
+Wire Wire Line
+	8050 1950 8050 3975
+Wire Wire Line
+	8050 3975 7525 3975
+Text Label 7950 1950 3    50   ~ 0
+d1'
+Text Label 7850 1950 3    50   ~ 0
+d4'
+Text Label 8050 1950 3    50   ~ 0
+~BUSRQ
+Text Notes 9625 2650 2    50   ~ 0
+TODO: ø1
+Text Notes 9625 2550 2    50   ~ 0
+TODO: 7M
+Text Label 925  3625 2    50   ~ 0
+7M
+$Comp
+L power:GND #PWR0117
+U 1 1 6158CDE9
+P 9775 3050
+F 0 "#PWR0117" H 9775 2800 50  0001 C CNN
+F 1 "GND" H 9780 2877 50  0000 C CNN
+F 2 "" H 9775 3050 50  0001 C CNN
+F 3 "" H 9775 3050 50  0001 C CNN
+	1    9775 3050
+	1    0    0    -1
+$EndComp
+Wire Wire Line
+	9775 3050 9775 2950
+Text Notes 9625 2850 2    50   ~ 0
+TODO: U3
+Text Label 925  1825 2    50   ~ 0
+DMA_IN
+Text Label 9425 1325 2    50   ~ 0
+DMA_IN
+Text Label 10850 1325 0    50   ~ 0
+~BUSRQ
+Wire Wire Line
+	10275 1325 10850 1325
+Wire Wire Line
+	9675 1325 9425 1325
+Wire Wire Line
+	10500 1125 10500 1175
+Wire Wire Line
+	10500 1175 10225 1175
+Wire Wire Line
+	10225 1175 10225 850
+Wire Wire Line
+	10225 850  9575 850
+Wire Wire Line
+	9575 850  9575 1275
+Wire Wire Line
+	9575 1275 9675 1275
+Wire Wire Line
+	9675 1275 9675 1325
+Connection ~ 9675 1325
+Text Label 8550 1950 3    50   ~ 0
+d6'
 $EndSCHEMATC

Commit message: a couple 7474s added
Parts:
- added D?: LED, symbol Device:LED
- added R1: 2.2k, symbol Device:R_Small_US
- added R?: 680Ω, symbol Device:R_Small_US
- added U3: 74LS32, symbol 74xx:74LS32
- added U5, U6: 74LS74, symbol 74xx:74LS74
Connections:
- net labels added: PUP, R~W, ~IOSEL, ~RESET, ~Z80_RESET, ~Z80_WAIT
- wire segments 34 -> 51
- no-connect marks 0 -> 2
Other:
- note added: "TODO: Clock stuff into pin 11"
Changed lines of the file:
@@
 Text Label 8550 1950 3    50   ~ 0
 d6'
+Text Label 2525 6425 0    50   ~ 0
+~IOSEL
+Text Label 2525 3025 0    50   ~ 0
+R~W
+Text Label 1025 7100 2    50   ~ 0
+~IOSEL
+Text Label 1025 7300 2    50   ~ 0
+R~W
+$Comp
+L 74xx:74LS32 U3
+U 1 1 615868BF
+P 1325 7200
+F 0 "U3" H 1325 7525 50  0000 C CNN
+F 1 "74LS32" H 1325 7434 50  0000 C CNN
+F 2 "" H 1325 7200 50  0001 C CNN
+F 3 "http://www.ti.com/lit/gpn/sn74LS32" H 1325 7200 50  0001 C CNN
+	1    1325 7200
+	1    0    0    -1
+$EndComp
+$Comp
+L 74xx:74LS74 U5
+U 1 1 6158ADF5
+P 2125 7300
+F 0 "U5" H 2125 7781 50  0000 C CNN
+F 1 "74LS74" H 2125 7690 50  0000 C CNN
+F 2 "" H 2125 7300 50  0001 C CNN
+F 3 "74xx/74hc_hct74.pdf" H 2125 7300 50  0001 C CNN
+	1    2125 7300
+	1    0    0    -1
+$EndComp
+Wire Wire Line
+	1625 7200 1725 7200
+Wire Wire Line
+	1725 7200 1725 7300
+Wire Wire Line
+	1725 7300 1825 7300
+$Comp
+L Device:LED D?
+U 1 1 6158DEE0
+P 625 7275
+F 0 "D?" V 664 7158 50  0000 R CNN
+F 1 "LED" V 573 7158 50  0000 R CNN
+F 2 "" H 625 7275 50  0001 C CNN
+F 3 "~" H 625 7275 50  0001 C CNN
+	1    625  7275
+	0    -1   -1   0
+$EndComp
+$Comp
+L Device:R_Small_US R?
+U 1 1 6158FB15
+P 625 7525
+F 0 "R?" H 693 7571 50  0000 L CNN
+F 1 "680Ω" H 693 7480 50  0000 L CNN
+F 2 "" H 625 7525 50  0001 C CNN
+F 3 "~" H 625 7525 50  0001 C CNN
+	1    625  7525
+	1    0    0    -1
+$EndComp
+$Comp
+L power:+5V #PWR?
+U 1 1 615905F5
+P 625 7125
+F 0 "#PWR?" H 625 6975 50  0001 C CNN
+F 1 "+5V" H 640 7298 50  0000 C CNN
+F 2 "" H 625 7125 50  0001 C CNN
+F 3 "" H 625 7125 50  0001 C CNN
+	1    625  7125
+	1    0    0    -1
+$EndComp
+Wire Wire Line
+	1775 7200 1825 7200
+$Comp
+L 74xx:74LS74 U5
+U 2 1 615927B0
+P 2925 7300
+F 0 "U5" H 2925 7781 50  0000 C CNN
+F 1 "74LS74" H 2925 7690 50  0000 C CNN
+F 2 "" H 2925 7300 50  0001 C CNN
+F 3 "74xx/74hc_hct74.pdf" H 2925 7300 50  0001 C CNN
+	2    2925 7300
+	1    0    0    -1
+$EndComp
+Wire Wire Line
+	2625 7200 2525 7200
+Wire Wire Line
+	2525 7200 2525 7600
+Wire Wire Line
+	2525 7600 2925 7600
+Connection ~ 2525 7200
+Wire Wire Line
+	2525 7200 2425 7200
+Wire Wire Line
+	2925 7000 2125 7000
+Connection ~ 2125 7000
+$Comp
+L Device:R_Small_US R1
+U 1 1 615970D2
+P 1675 6900
+F 0 "R1" H 1743 6946 50  0000 L CNN
+F 1 "2.2k" H 1743 6855 50  0000 L CNN
+F 2 "" H 1675 6900 50  0001 C CNN
+F 3 "~" H 1675 6900 50  0001 C CNN
+	1    1675 6900
+	1    0    0    -1
+$EndComp
+Wire Wire Line
+	1675 7000 2125 7000
+$Comp
+L power:+5V #PWR?
+U 1 1 61599033
+P 1675 6800
+F 0 "#PWR?" H 1675 6650 50  0001 C CNN
+F 1 "+5V" H 1690 6973 50  0000 C CNN
+F 2 "" H 1675 6800 50  0001 C CNN
+F 3 "" H 1675 6800 50  0001 C CNN
+	1    1675 6800
+	1    0    0    -1
+$EndComp
+Text Label 1975 7000 1    50   ~ 0
+PUP
+Wire Wire Line
+	625  7625 625  7700
+Wire Wire Line
+	625  7700 1775 7700
+Wire Wire Line
+	2425 7700 2425 7400
+Wire Wire Line
+	1775 7200 1775 7700
+Connection ~ 1775 7700
+Wire Wire Line
+	1775 7700 2425 7700
+Text Label 925  2625 2    50   ~ 0
+~RESET
+$Comp
+L 74xx:74LS74 U6
+U 1 1 615A74E8
+P 1150 9325
+F 0 "U6" H 1150 9806 50  0000 C CNN
+F 1 "74LS74" H 1150 9715 50  0000 C CNN
+F 2 "" H 1150 9325 50  0001 C CNN
+F 3 "74xx/74hc_hct74.pdf" H 1150 9325 50  0001 C CNN
+	1    1150 9325
+	1    0    0    -1
+$EndComp
+Text Label 850  8875 2    50   ~ 0
+PUP
+Wire Wire Line
+	850  8875 850  9025
+Wire Wire Line
+	850  9025 1150 9025
+Text Label 850  9225 2    50   ~ 0
+~RESET
+Text Label 1450 9225 0    50   ~ 0
+~Z80_RESET
+Text Label 7525 4075 0    50   ~ 0
+~Z80_RESET
+Text Label 1150 9625 3    50   ~ 0
+PUP
+NoConn ~ 1450 9425
+Text Label 3225 7200 0    50   ~ 0
+~Z80_WAIT
+Text Label 7525 3875 0    50   ~ 0
+~Z80_WAIT
+NoConn ~ 3225 7400
+Text Notes 2525 7750 0    50   ~ 0
+TODO: Clock stuff into pin 11
 $EndSCHEMATC

Commit message: More ICs placed
Parts:
- added U1: 74LS00, Package_DIP:DIP-14_W7.62mm, symbol 74xx:74LS00
- added unit 4 of U3
- added unit 2 of U3
- added unit 2 of U6
- D1: renamed from D?; footprint (none) -> LED_THT:LED_D5.0mm
- R1: footprint (none) -> Resistor_THT:R_Axial_DIN0207_L6.3mm_D2.5mm_P7.62mm_Horizontal
- R8: renamed from R?; footprint (none) -> Resistor_THT:R_Axial_DIN0207_L6.3mm_D2.5mm_P7.62mm_Horizontal
- U3, U5, U6: footprint (none) -> Package_DIP:DIP-14_W7.62mm
Connections:
- net labels added: RW_OUT, Z80_RW
- wire segments 51 -> 76
- no-connect marks 2 -> 7
