File: a2card_template.kicad_pcb (KiCad board)
At the start: 2 copper layers, 158.8 x 76.4 mm, 19 parts, among them U1 74LS00, U10 PLCCZ80, U14 74LS367, U15 74LS373, U16 74LS367, U17 74LS367, U3 74LS32, U5 74LS74, U6 74LS74, U7 74LS86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

Commit message: KiCad Upgrade
Connections:
- net /R~W renamed /R~{W}
- net /~BUSRQ renamed /~{BUSRQ}
- net /~IOSEL renamed /~{IOSEL}
- net /~IRQ renamed /~{IRQ}
- net /~NMI renamed /~{NMI}
- net /~RD renamed /~{RD}
- net /~RESET renamed /~{RESET}
- net /~Z80_IRQ renamed /~{Z80_IRQ}
- net /~Z80_NMI renamed /~{Z80_NMI}
- net /~Z80_RESET renamed /~{Z80_RESET}
- net /~Z80_WAIT renamed /~{Z80_WAIT}
Other:
- net class Default removed
